File: Eagle/ENGI301 Project Actual.brd (EAGLE design)
At the start: 152.4 x 63.5 mm, 31 parts, among them U1 POCKETBEAGLE, U2 MOD-LED8X8RGB-CONN, U3 MOD-LED8X8RGB-CONN

Commit message: THIS IS THE REAL FINAL ONE - PALMER
Sorry for this mess of a gitHub
Parts:
- moved R2 4.06 mm to (128.8, 40.4)
Routing:
- net I2C2.SDA: track 127.7 -> 131.8 mm
- net SYS_VDD1_3P3V: track 254.3 -> 258.4 mm
Changed lines of the file:
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@@
 <element name="C3" library="ENGI301 Project 2a" package="C0603" value="0.1uF" x="147.832" y="19.166" rot="R180"/>
 <element name="R1" library="ENGI301 Project 2a" package="R0603" value="2.2k" x="134.832" y="25.936"/>
-<element name="R2" library="ENGI301 Project 2a" package="R0603" value="2.2k" x="128.796" y="36.298"/>
+<element name="R2" library="ENGI301 Project 2a" package="R0603" value="2.2k" x="128.796" y="40.362"/>
 <element name="R3" library="ENGI301 Project 2a" package="R0603" value="1k" x="124.06" y="24.33"/>
 <element name="R4" library="ENGI301 Project 2a" package="R0603" value="1k" x="124.25" y="19.25"/>
@@
 <wire x1="129.54" y1="34.671" x2="129.54" y2="36.195" width="0.127" layer="1"/>
 <wire x1="128.524" y1="32.512" x2="129.54" y2="33.528" width="0.127" layer="1"/>
-<wire x1="129.54" y1="36.195" x2="129.5961" y2="36.298" width="0.127" layer="1"/>
+<wire x1="129.54" y1="36.195" x2="129.5961" y2="40.362" width="0.127" layer="1"/>
 <wire x1="146.05" y1="29.718" x2="145.796" y2="29.718" width="0.127" layer="1"/>
 <wire x1="146.304" y1="29.972" x2="146.05" y2="29.718" width="0.127" layer="1"/>
@@
 <wire x1="128.016" y1="36.195" x2="128.778" y2="35.433" width="0.127" layer="1"/>
 <wire x1="143.129" y1="32.258" x2="143.2" y2="32.21" width="0.127" layer="1"/>
-<wire x1="128.016" y1="36.195" x2="127.9959" y2="36.298" width="0.127" layer="1"/>
+<wire x1="128.016" y1="36.195" x2="127.9959" y2="40.362" width="0.127" layer="1"/>
 <wire x1="39.243" y1="8.255" x2="37.973" y2="8.255" width="0.127" layer="16"/>
 <wire x1="42.545" y1="11.557" x2="39.243" y2="8.255" width="0.127" layer="16"/>
