File: Eagle/ENGI301 Project Actual.sch (EAGLE design)
At the start: 27 parts, among them U1 POCKETBEAGLE, U2 MOD-LED8X8RGB-CONN, U3 MOD-LED8X8RGB-CONN

Commit message: THIS IS THE REAL FINAL ONE - PALMER
Sorry for this mess of a gitHub
Changed lines of the file:
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@@
 <instance part="GND10" gate="1" x="299.72" y="50.8"/>
 <instance part="GND11" gate="1" x="200.66" y="165.1"/>
-<instance part="GND12" gate="1" x="134.62" y="167.64"/>
+<instance part="GND12" gate="1" x="134.62" y="170.18"/>
 <instance part="GND13" gate="1" x="111.76" y="116.84"/>
 <instance part="GND14" gate="1" x="48.26" y="99.06"/>
@@
 <pinref part="GND12" gate="1" pin="GND"/>
 <wire x1="139.7" y1="175.26" x2="134.62" y2="175.26" width="0.1524" layer="91"/>
-<wire x1="134.62" y1="175.26" x2="134.62" y2="170.18" width="0.1524" layer="91"/>
+<wire x1="134.62" y1="175.26" x2="134.62" y2="172.72" width="0.1524" layer="91"/>
 </segment>
 <segment>
